File: bmw-obc-backlight.sch (KiCad schematic (older format))
At the start: 4 parts, among them J1 Conn_01x02

Commit message: Swapped resistor to SMT. There isn't enough space for a through hole unless it's between the LED legs.
Parts:
- R1: footprint Resistor_THT:R_Axial_DIN0207_L6.3mm_D2.5mm_P10.16mm_Horizontal -> Resistor_SMD:R_1206_3216Metric_Pad1.30x1.75mm_HandSolder
Changed lines of the file:
@@
 F 0 "R1" H 820 1096 50  0000 L CNN
 F 1 "10000" H 820 1005 50  0000 L CNN
-F 2 "Resistor_THT:R_Axial_DIN0207_L6.3mm_D2.5mm_P10.16mm_Horizontal" V 680 1050 50  0001 C CNN
+F 2 "Resistor_SMD:R_1206_3216Metric_Pad1.30x1.75mm_HandSolder" V 680 1050 50  0001 C CNN
 F 3 "https://page.venkel.com/hubfs/Resources/Datasheets/CR-Series.pdf" H 750 1050 50  0001 C CNN
 F 4 "https://page.venkel.com/hubfs/Resources/Datasheets/CR-Series.pdf" H 750 1050 50  0001 C CNN "SMT Equiv"

Commit message: Swap to surface mount LEDs and add JLC manufacturing information
Parts:
- D1, D2: footprint LED_THT:LED_D5.0mm -> LED_SMD:LED_0805_2012Metric_Castellated; symbol Device:LED -> bmw-obc-backlight-rescue:LED-Device; JLC (none) -> 0805; LCSC (none) -> C2293
- J1: symbol Connector_Generic:Conn_01x02 -> bmw-obc-backlight-rescue:Conn_01x02-Connector_Generic
- R1: symbol Device:R -> bmw-obc-backlight-rescue:R-Device; JLC (none) -> 1206; LCSC (none) -> C17902
Changed lines of the file:
@@
 $EndDescr
 $Comp
-L Connector_Generic:Conn_01x02 J1
+L bmw-obc-backlight-rescue:Conn_01x02-Connector_Generic J1
 U 1 1 60235A24
 P 1650 1000
@@
 $EndComp
 $Comp
-L Device:LED D1
+L bmw-obc-backlight-rescue:LED-Device D1
 U 1 1 6023A561
 P 1050 750
 F 0 "D1" H 1043 967 50  0000 C CNN
 F 1 "LED" H 1043 876 50  0000 C CNN
-F 2 "LED_THT:LED_D5.0mm" H 1050 750 50  0001 C CNN
+F 2 "LED_SMD:LED_0805_2012Metric_Castellated" H 1050 750 50  0001 C CNN
 F 3 "~" H 1050 750 50  0001 C CNN
+F 4 "0805" H 1050 750 50  0001 C CNN "JLC"
+F 5 "C2293" H 1050 750 50  0001 C CNN "LCSC"
 	1    1050 750
 	1    0    0    -1
@@
 	1350 1000 1350 750
 $Comp
-L Device:LED D2
+L bmw-obc-backlight-rescue:LED-Device D2
 U 1 1 6023B59A
 P 1050 1350
 F 0 "D2" H 1050 1550 50  0000 C CNN
 F 1 "LED" H 1050 1450 50  0000 C CNN
-F 2 "LED_THT:LED_D5.0mm" H 1050 1350 50  0001 C CNN
+F 2 "LED_SMD:LED_0805_2012Metric_Castellated" H 1050 1350 50  0001 C CNN
 F 3 "~" H 1050 1350 50  0001 C CNN
+F 4 "0805" H 1050 1350 50  0001 C CNN "JLC"
+F 5 "C2293" H 1050 1350 50  0001 C CNN "LCSC"
 	1    1050 1350
 	-1   0    0    1
 $EndComp
 $Comp
-L Device:R R1
+L bmw-obc-backlight-rescue:R-Device R1
 U 1 1 60238D1F
 P 750 1050
@@
 F 3 "https://page.venkel.com/hubfs/Resources/Datasheets/CR-Series.pdf" H 750 1050 50  0001 C CNN
 F 4 "https://page.venkel.com/hubfs/Resources/Datasheets/CR-Series.pdf" H 750 1050 50  0001 C CNN "SMT Equiv"
+F 5 "1206" H 750 1050 50  0001 C CNN "JLC"
+F 6 "C17902" H 750 1050 50  0001 C CNN "LCSC"
 	1    750  1050
 	1    0    0    -1

Commit message: Changes for ordering
Parts:
- J1: Spice_Model (none) -> dc 12; Spice_Netlist_Enabled (none) -> Y; Spice_Primitive (none) -> V
Changed lines of the file:
@@
 F 2 "bmw-obc-backlight-footprints:TE_2Position_2.54mmPitch_Horizontal_Header" H 1650 1000 50  0001 C CNN
 F 3 "https://media.digikey.com/pdf/Data%20Sheets/Tyco%20Electonics%20AMP%20PDFs/535676.pdf" H 1650 1000 50  0001 C CNN
+F 4 "V" H 1650 1000 50  0001 C CNN "Spice_Primitive"
+F 5 "dc 12" H 1650 1000 50  0001 C CNN "Spice_Model"
+F 6 "Y" H 1650 1000 50  0001 C CNN "Spice_Netlist_Enabled"
 	1    1650 1000
 	1    0    0    -1

Commit message: Update LED part number to white LED
Parts:
- D1: LCSC C2293 -> C34499
Changed lines of the file:
@@
 F 3 "~" H 1050 750 50  0001 C CNN
 F 4 "0805" H 1050 750 50  0001 C CNN "JLC"
-F 5 "C2293" H 1050 750 50  0001 C CNN "LCSC"
+F 5 "C34499" H 1050 750 50  0001 C CNN "LCSC"
 	1    1050 750
 	1    0    0    -1
